Commit message: ros-robot pkg update xacro files accroding to the new configuration of the laser

File: xacros/microEpsilon30x25.xacro (robot description, xacro)
@@ -21,6 +21,9 @@
         <!-- <origin xyz="-0.057 0.057 0.106" rpy="-1.5707963 0 -0.785398"/>  -->
         <!-- <origin xyz="-0.007775734219481385 0.07877175919435352 0.07711115615836664" rpy="-1.560126692578499 -0.001809474317625123 -1.4"/>  -->
-        <origin xyz="0.209 0 0.1285" rpy="-1.560126692578499 -0.001809474317625123 -1.5708"/>  <!-- Estimated Points 22-9-2024 -->
-        <origin xyz="0.167435263 0 0.094955992" rpy="-1.586489371353562161 -0.001794942 -1.580455807991475226"/>  <!-- Calibrated Points 22-9-2024 -->
+        <!--<origin xyz="0.209 0 0.1285" rpy="-1.560126692578499 -0.001809474317625123 -1.5708"/>  --><!-- Estimated Points 22-9-2024 -->
+        <!-- calibration at aric blue laser -->
+        <!-- <origin xyz="0.167435263 0 0.094955992" rpy="-1.586489371353562161 -0.001794942 -1.580455807991475226"/>  Calibrated Points 22-9-2024 -->
+        <!-- calibration at sanad blue laser 22-12-2025 -->
+        <origin xyz="-0.16831833020587256 0 0.0931629563611275" rpy="-1.5702677795327937 0 1.5714674315073291"/>  <!-- Calibrated Points 22-9-2024 -->
     </joint>
     <joint name="exact_laser_transform" type="fixed">
